File: pixel_qi_button_boards.kicad_pcb (KiCad board)
At the start: 2 copper layers, 19 parts, among them J1 Conn_01x08, J2 Conn_01x06, J3 Conn_01x06, SW1 B3SE, SW10 B3SE, SW11 B3SE, SW12 B3SE, SW13 B3SE, SW14 B3SE, SW15 B3SE, SW16 B3SE, SW2 B3SE, SW3 B3SE, SW4 B3SE, SW5 B3SE, SW6 B3SE, SW7 B3SE, SW8 B3SE, SW9 B3SE

Commit message: Finished pcb layout
Parts:
- removed J3: Conn_01x06, Connectors_Molex:Molex_PicoBlade_53398-0671_06x1.25mm_Straight
- removed SW12, SW13, SW14, SW15, SW16: B3SE, Buttons_Switches_SMD:SW_SPST_B3SL-1002P
- added REF1: MountingHole_2.2mm_M2, Mounting_Holes:MountingHole_2.2mm_M2, F.Cu at (49.1, 115.3)
- added REF10: MountingHole_2.2mm_M2, Mounting_Holes:MountingHole_2.2mm_M2, F.Cu at (134.8, 141.7)
- added REF11: MountingHole_2.2mm_M2, Mounting_Holes:MountingHole_2.2mm_M2, F.Cu at (158.6, 141.7)
- added REF12: MountingHole_2.2mm_M2, Mounting_Holes:MountingHole_2.2mm_M2, F.Cu at (182.4, 141.7)
- added REF13: MountingHole_2.2mm_M2, Mounting_Holes:MountingHole_2.2mm_M2, F.Cu at (206.2, 141.7)
- added REF2: MountingHole_2.2mm_M2, Mounting_Holes:MountingHole_2.2mm_M2, F.Cu at (82.5, 115.3)
- added REF3: MountingHole_2.2mm_M2, Mounting_Holes:MountingHole_2.2mm_M2, F.Cu at (116.0, 115.3)
- added REF4: MountingHole_2.2mm_M2, Mounting_Holes:MountingHole_2.2mm_M2, F.Cu at (149.4, 115.3)
- added REF5: MountingHole_2.2mm_M2, Mounting_Holes:MountingHole_2.2mm_M2, F.Cu at (182.8, 115.3)
- added REF6: MountingHole_2.2mm_M2, Mounting_Holes:MountingHole_2.2mm_M2, F.Cu at (216.3, 115.3)
- added REF7: MountingHole_2.2mm_M2, Mounting_Holes:MountingHole_2.2mm_M2, F.Cu at (249.7, 115.3)
- added REF8: MountingHole_2.2mm_M2, Mounting_Holes:MountingHole_2.2mm_M2, F.Cu at (87.1, 141.7)
- added REF9: MountingHole_2.2mm_M2, Mounting_Holes:MountingHole_2.2mm_M2, F.Cu at (110.9, 141.7)
- J1: value Conn_01x08 -> Conn_01x07; footprint Connectors_Molex:Molex_PicoBlade_53398-0871_08x1.25mm_Straight -> Connectors_Hirose:Hirose_DF13C-07P-1.25V_07x1.25mm_Straight; moved to B.Cu
- J2: footprint Connectors_Molex:Molex_PicoBlade_53398-0671_06x1.25mm_Straight -> Connectors_Hirose:Hirose_DF13C-06P-1.25V_06x1.25mm_Straight; moved to B.Cu
- moved SW6 67.6 mm to (233.0, 115.3)
- moved J1 55.4 mm to (132.7, 115.7)
- moved SW5 49.1 mm to (199.6, 115.3)
- moved SW11 48.3 mm to (194.3, 141.7)
- moved SW10 38.5 mm to (170.5, 141.7)
- moved SW1 31.7 mm to (65.8, 115.3)
- moved SW4 31.3 mm to (166.2, 115.3)
- moved SW9 27.8 mm to (146.7, 141.7)
- moved J2 23.9 mm to (146.7, 142.1)
- moved SW8 16.3 mm to (122.8, 141.7)
- moved SW2 15.8 mm to (99.2, 115.3)
- moved SW3 15.2 mm to (132.7, 115.3)
- moved SW7 6.20 mm to (99.0, 141.7)
Connections:
- SW1 pad 1: Net-(J1-Pad1) -> Net-(J1-Pad4)
- SW1 pad 2: Net-(J1-Pad7) -> Net-(J1-Pad1)
- SW10 pad 1: Net-(J2-Pad1) -> Net-(J2-Pad4)
- SW10 pad 2: Net-(J2-Pad4) -> Net-(J2-Pad5)
- SW11 pad 1: Net-(J2-Pad1) -> Net-(J2-Pad4)
- SW11 pad 2: Net-(J2-Pad3) -> Net-(J2-Pad6)
- SW2 pad 1: Net-(J1-Pad1) -> Net-(J1-Pad4)
- SW2 pad 2: Net-(J1-Pad6) -> Net-(J1-Pad2)
- SW3 pad 1: Net-(J1-Pad1) -> Net-(J1-Pad4)
- SW3 pad 2: Net-(J1-Pad5) -> Net-(J1-Pad3)
- SW4 pad 1: Net-(J1-Pad1) -> Net-(J1-Pad4)
- SW4 pad 2: Net-(J1-Pad4) -> Net-(J1-Pad5)
- SW5 pad 1: Net-(J1-Pad1) -> Net-(J1-Pad4)
- SW5 pad 2: Net-(J1-Pad3) -> Net-(J1-Pad6)
- SW6 pad 1: Net-(J1-Pad1) -> Net-(J1-Pad4)
- SW6 pad 2: Net-(J1-Pad2) -> Net-(J1-Pad7)
- SW7 pad 1: Net-(J2-Pad1) -> Net-(J2-Pad4)
- SW7 pad 2: Net-(J2-Pad2) -> Net-(J2-Pad1)
- SW8 pad 1: Net-(J2-Pad1) -> Net-(J2-Pad4)
- SW8 pad 2: Net-(J2-Pad6) -> Net-(J2-Pad2)
- SW9 pad 1: Net-(J2-Pad1) -> Net-(J2-Pad4)
- SW9 pad 2: Net-(J2-Pad5) -> Net-(J2-Pad3)
Routing:
- net Net-(J1-Pad4): track 0.00 -> 183.3 mm, vias 0 -> 1
- net Net-(J2-Pad4): track 0.00 -> 110.7 mm, vias 0 -> 1
- net Net-(J1-Pad7): track 0.00 -> 100.4 mm, vias 0 -> 1
- net Net-(J1-Pad6): track 0.00 -> 70.0 mm, vias 0 -> 1
- net Net-(J1-Pad1): track 0.00 -> 66.9 mm, vias 0 -> 1
- net Net-(J2-Pad6): track 0.00 -> 48.7 mm, vias 0 -> 1
- net Net-(J2-Pad1): track 0.00 -> 48.4 mm, vias 0 -> 1
- net Net-(J1-Pad5): track 0.00 -> 38.4 mm, vias 0 -> 1
- net Net-(J1-Pad2): track 0.00 -> 36.3 mm, vias 0 -> 1
- net Net-(J2-Pad5): track 0.00 -> 27.7 mm, vias 0 -> 1
- net Net-(J2-Pad2): track 0.00 -> 27.4 mm, vias 0 -> 1
- net Net-(J1-Pad3): track 0.00 -> 11.2 mm, vias 0 -> 1
- net Net-(J2-Pad3): track 0.00 -> 11.1 mm, vias 0 -> 1
Other:
- board outline added: 208.5 x 36.4 mm
- rule pad_to_mask_clearance: 0.2 -> 0.0508

Commit message: Added label to board
Other:
- board text added: "bit-builder.com/pixel_qi_button_boards-v1.1"
Changed lines of the file:
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@@
     (area 39.592857 109.825 259.257143 147.525)
     (thickness 1.6)
-    (drawings 9)
+    (drawings 11)
     (tracks 119)
     (zones 0)
@@
   (title_block
     (title "Pixel Qi Button Board PCB")
-    (rev 1)
+    (rev 1.1)
   )
   (layers
@@
     )
   )
+  (gr_text bit-builder.com/pixel_qi_button_boards-v1.1 (at 110.5 145.3) (layer B.SilkS)
+    (effects (font (size 1.5 1.5) (thickness 0.3)) (justify mirror))
+  )
+  (gr_text bit-builder.com/pixel_qi_button_boards-v1.1 (at 72.4 119) (layer B.SilkS)
+    (effects (font (size 1.5 1.5) (thickness 0.3)) (justify mirror))
+  )
   (gr_line (start 83 136.7) (end 83.05 136.7) (angle 90) (layer Edge.Cuts) (width 0.15))
